File: PCV MATOME MAIN V5-KICAD 5.0/PCV MATOME MAIN V5-KICAD 5.0.sch (KiCad schematic (older format))
At the start: 41 parts, among them P1 Digital, P10 CONN_01X01, P11 CONN_01X01, P12 CONN_01X01, P13 CONN_01X01, P2 Power, P3 Analog, P4 Analog, P5 PWM, P6 PWM, P7 Communication, P8 CONN_01X01, P9 CONN_01X01, U1 ESP-12F

Commit message: mofifile 08012018
Parts:
- removed J?: Conn_01x04, symbol Connector_Generic:Conn_01x04
- added C? (x4): 100n, symbol Device:C
- added C? (x2): 100n, symbol pspice:CAP
- added J?: Conn_01x02, symbol Connector_Generic:Conn_01x02
- added J?: Conn_01x08, symbol Connector_Generic:Conn_01x08
- added J? (x2): Conn_02x08_Odd_Even, symbol Connector_Generic:Conn_02x08_Odd_Even
- added J?: Conn_02x06_Top_Bottom, symbol Connector_Generic:Conn_02x06_Top_Bottom
- added R? (x6): 10K, symbol Device:R
- added U? (x2): MAX7219, symbol max:MAX7219
Connections:
- net labels added: 1-C1, 1-C2, 1-C3, 1-C4, 1-C5, 1-C6, 1-C7, 1-C8, 1-R1, 1-R2, 1-R3, 1-R4, 1-R5, 1-R6, 1-R7, 1-R8, 2-C1, 2-C2, 2-C3, 2-C4, 2-C5, 2-C6, 2-C7, 2-C8, 2-R1, 2-R2, 2-R3, 2-R4, 2-R5, 2-R6, 2-R7, 2-R8, BACK, CLK_M, DIN_M, HOME, NEXT, SC_M, SET
- net labels removed: RXD, TXD
- wire segments 214 -> 356
- no-connect marks 24 -> 25

Commit message: finish schematic
Parts:
- removed C? (x4): 100n, symbol Device:C
- added C10, C11, C12, C13, C14, C15, C16, C17, C18, C19, C20, C21, C22, C23, C24, C5, C6, C7, C8, C9: 100n, symbol Device:C_Small
- added C26: 10u, symbol Device:CP
- added C28: 100u, symbol Device:CP
- added D1, D3, D4: D, symbol Device:D
- added J11: Conn_01x04, symbol Connector_Generic:Conn_01x04
- added J13, J8: Conn_01x08, symbol Connector_Generic:Conn_01x08
- added J15: Conn_01x02, symbol Connector_Generic:Conn_01x02
- added J9: Conn_01x16, symbol Connector_Generic:Conn_01x16
- added R18: 100, symbol Device:R
- added RN1, RN2: R_Network08, Resistor_THT:R_Array_SIP9, symbol Device:R_Network08
- added RV1: R_POT, symbol Device:R_POT
- added U5: LD1117S50TR_SOT223, Package_TO_SOT_SMD:SOT-223-3_TabPin2, symbol Regulator_Linear:LD1117S50TR_SOT223
- gave numbers to parts that had none: 41
Connections:
- net labels added: D4, D5, D6, D7, EN, GNDPWR, RS, RW, SW1, SW10, SW11, SW12, SW13, SW14, SW15, SW16, SW2, SW3, SW4, SW5, SW6, SW7, SW8, SW9
- wire segments 356 -> 527
- no-connect marks 25 -> 66
Other:
- moved on the sheet: U4

Commit message: finish schematic
Parts:
- C1, C10, C11, C12, C13, C14, C15, C16, C17, C18, C19, C2, C20, C21, C22, C23, C24, C25, C3, C4, C5, C6, C7, C8, C9: footprint (none) -> Capacitor_SMD:C_0805_2012Metric_Pad1.15x1.40mm_HandSolder
- C26: footprint (none) -> Capacitor_SMD:CP_Elec_4x5.4
- C27, C28: footprint (none) -> Capacitor_SMD:CP_Elec_8x6.5
- D1, D2, D3, D4: footprint (none) -> Diode_SMD:D_SOD-123
- J1, J2: footprint (none) -> Connector_IDC:IDC-Header_2x08_P2.54mm_Horizontal
- J10: footprint (none) -> Connector_JST:JST_EH_S02B-EH_1x02_P2.50mm_Horizontal
- J11: footprint (none) -> Connector_JST:JST_EH_S04B-EH_1x04_P2.50mm_Horizontal
- J12, J13, J8: footprint (none) -> Connector_JST:JST_EH_S08B-EH_1x08_P2.50mm_Horizontal
- J14, J15: footprint (none) -> Connector_Wire:SolderWirePad_1x02_P5.08mm_Drill1.5mm
- J3, J4, J6, J7: footprint (none) -> Connector_JST:JST_EH_S06B-EH_1x06_P2.50mm_Horizontal
- J9: footprint (none) -> Connector_JST:JST_EH_S16B-EH_1x16_P2.50mm_Horizontal
- R1, R10, R11, R12, R13, R14, R15, R16, R17, R18, R2, R3, R4, R5, R6, R7, R8, R9: footprint (none) -> Resistor_SMD:R_0805_2012Metric_Pad1.15x1.40mm_HandSolder
- RV1: footprint (none) -> Potentiometer_THT:Potentiometer_Bourns_3296W_Vertical
- U2, U3: footprint (none) -> Package_SO:SOIC-24W_7.5x15.4mm_P1.27mm
- U4: footprint (none) -> Package_TO_SOT_SMD:SOT-223-3_TabPin2
- U5: footprint Package_TO_SOT_SMD:SOT-223-3_TabPin2 -> Package_TO_SOT_THT:TO-220-3_Vertical
Connections:
- wire segments 527 -> 531

Commit message: initinal pcb
Parts:
- removed J5: Conn_02x06_Top_Bottom, symbol Connector_Generic:Conn_02x06_Top_Bottom
- added U6: SHIFT_LEVEL_3.3V_5V, LEEVAWNS:SHIFTLEVEL, symbol LEEVAWNS:SHIFT_LEVEL_3.3V_5V
- J1, J2: footprint Connector_IDC:IDC-Header_2x08_P2.54mm_Horizontal -> Connector_IDC:IDC-Header_2x08_P2.54mm_Vertical
- J10: footprint Connector_JST:JST_EH_S02B-EH_1x02_P2.50mm_Horizontal -> Connector_JST:JST_EH_B02B-EH-A_1x02_P2.50mm_Vertical
- J11: footprint Connector_JST:JST_EH_S04B-EH_1x04_P2.50mm_Horizontal -> Connector_JST:JST_EH_B04B-EH-A_1x04_P2.50mm_Vertical
- J12, J13, J8: footprint Connector_JST:JST_EH_S08B-EH_1x08_P2.50mm_Horizontal -> Connector_JST:JST_EH_B08B-EH-A_1x08_P2.50mm_Vertical
- J3, J4, J6, J7: footprint Connector_JST:JST_EH_S06B-EH_1x06_P2.50mm_Horizontal -> Connector_JST:JST_EH_B06B-EH-A_1x06_P2.50mm_Vertical
- J9: footprint Connector_JST:JST_EH_S16B-EH_1x16_P2.50mm_Horizontal -> Connector_JST:JST_EH_B16B-EH-A_1x16_P2.50mm_Vertical
- SW1: footprint (none) -> Button_Switch_THT:SW_DIP_SPSTx01_Slide_9.78x4.72mm_W7.62mm_P2.54mm
Changed lines of the file:
@@
 F 0 "SW1" H 950 1935 50  0000 C CNN
 F 1 "SW_Push" H 950 1844 50  0000 C CNN
-F 2 "" H 950 1850 50  0001 C CNN
+F 2 "Button_Switch_THT:SW_DIP_SPSTx01_Slide_9.78x4.72mm_W7.62mm_P2.54mm" H 950 1850 50  0001 C CNN
 F 3 "" H 950 1850 50  0001 C CNN
 	1    950  1650
@@
 F 0 "J3" H 6030 6242 50  0000 L CNN
 F 1 "Conn_01x06" H 6030 6151 50  0000 L CNN
-F 2 "Connector_JST:JST_EH_S06B-EH_1x06_P2.50mm_Horizontal" H 5950 6250 50  0001 C CNN
+F 2 "Connector_JST:JST_EH_B06B-EH-A_1x06_P2.50mm_Vertical" H 5950 6250 50  0001 C CNN
 F 3 "~" H 5950 6250 50  0001 C CNN
 	1    5950 6250
@@
 F 0 "J6" H 7280 6242 50  0000 L CNN
 F 1 "Conn_01x06" H 7280 6151 50  0000 L CNN
-F 2 "Connector_JST:JST_EH_S06B-EH_1x06_P2.50mm_Horizontal" H 7200 6250 50  0001 C CNN
+F 2 "Connector_JST:JST_EH_B06B-EH-A_1x06_P2.50mm_Vertical" H 7200 6250 50  0001 C CNN
 F 3 "~" H 7200 6250 50  0001 C CNN
 	1    7200 6250
@@
 F 0 "J4" H 6030 7092 50  0000 L CNN
 F 1 "Conn_01x06" H 6030 7001 50  0000 L CNN
-F 2 "Connector_JST:JST_EH_S06B-EH_1x06_P2.50mm_Horizontal" H 5950 7100 50  0001 C CNN
+F 2 "Connector_JST:JST_EH_B06B-EH-A_1x06_P2.50mm_Vertical" H 5950 7100 50  0001 C CNN
 F 3 "~" H 5950 7100 50  0001 C CNN
 	1    5950 7100
@@
 F 0 "J7" H 7280 7092 50  0000 L CNN
 F 1 "Conn_01x06" H 7280 7001 50  0000 L CNN
-F 2 "Connector_JST:JST_EH_S06B-EH_1x06_P2.50mm_Horizontal" H 7200 7100 50  0001 C CNN
+F 2 "Connector_JST:JST_EH_B06B-EH-A_1x06_P2.50mm_Vertical" H 7200 7100 50  0001 C CNN
 F 3 "~" H 7200 7100 50  0001 C CNN
 	1    7200 7100
@@
 F 0 "J10" H 10630 2692 50  0000 L CNN
 F 1 "Conn_01x02" H 10630 2601 50  0000 L CNN
-F 2 "Connector_JST:JST_EH_S02B-EH_1x02_P2.50mm_Horizontal" H 10550 2700 50  0001 C CNN
+F 2 "Connector_JST:JST_EH_B02B-EH-A_1x02_P2.50mm_Vertical" H 10550 2700 50  0001 C CNN
 F 3 "~" H 10550 2700 50  0001 C CNN
 	1    10550 2700
@@
 F 0 "J12" H 11700 1200 50  0000 L CNN
 F 1 "Conn_01x08" H 11700 1100 50  0000 L CNN
-F 2 "Connector_JST:JST_EH_S08B-EH_1x08_P2.50mm_Horizontal" H 12000 1700 50  0001 C CNN
+F 2 "Connector_JST:JST_EH_B08B-EH-A_1x08_P2.50mm_Vertical" H 12000 1700 50  0001 C CNN
 F 3 "~" H 12000 1700 50  0001 C CNN
 	1    12000 1700
@@
 F 0 "J1" H 2150 7317 50  0000 C CNN
 F 1 "Conn_02x08_Odd_Even" H 2150 7226 50  0000 C CNN
-F 2 "Connector_IDC:IDC-Header_2x08_P2.54mm_Horizontal" H 2100 6800 50  0001 C CNN
+F 2 "Connector_IDC:IDC-Header_2x08_P2.54mm_Vertical" H 2100 6800 50  0001 C CNN
 F 3 "~" H 2100 6800 50  0001 C CNN
 	1    2100 6800
@@
 F 0 "J2" H 3400 7317 50  0000 C CNN
 F 1 "Conn_02x08_Odd_Even" H 3400 7226 50  0000 C CNN
-F 2 "Connector_IDC:IDC-Header_2x08_P2.54mm_Horizontal" H 3350 6800 50  0001 C CNN
+F 2 "Connector_IDC:IDC-Header_2x08_P2.54mm_Vertical" H 3350 6800 50  0001 C CNN
 F 3 "~" H 3350 6800 50  0001 C CNN
 	1    3350 6800
@@
 Wire Wire Line
 	14850 4550 14850 4900
-$Comp
-L Connector_Generic:Conn_02x06_Top_Bottom J5
-U 1 1 5C1B7912
-P 5400 1600
-F 0 "J5" H 5450 2017 50  0000 C CNN
-F 1 "Conn_02x06_Top_Bottom" H 5450 1926 50  0000 C CNN
-F 2 "" H 5400 1600 50  0001 C CNN
-F 3 "~" H 5400 1600 50  0001 C CNN
-	1    5400 1600
-	1    0    0    -1
-$EndComp
 Text GLabel 5050 1200 1    50   Input ~ 0
 LV
-Text GLabel 5800 1200 1    50   Input ~ 0
+Text GLabel 6000 1200 1    50   Input ~ 0
 HV
 $Comp
@@
 L power:GND #PWR0130
 U 1 1 5C1B88F7
-P 5850 1500
-F 0 "#PWR0130" H 5850 1250 50  0001 C CNN
-F 1 "GND" H 5855 1327 50  0000 C CNN
-F 2 "" H 5850 1500 50  0001 C CNN
-F 3 "" H 5850 1500 50  0001 C CNN
-	1    5850 1500
+P 6050 1500
+F 0 "#PWR0130" H 6050 1250 50  0001 C CNN
+F 1 "GND" H 6055 1327 50  0000 C CNN
+F 2 "" H 6050 1500 50  0001 C CNN
+F 3 "" H 6050 1500 50  0001 C CNN
+	1    6050 1500
 	0    -1   -1   0
 $EndComp
 Wire Wire Line
-	5050 1400 5200 1400
-Wire Wire Line
 	5050 1200 5050 1400
 Wire Wire Line
-	5700 1400 5800 1400
-Wire Wire Line
-	5800 1400 5800 1200
-Wire Wire Line
-	5200 1500 5000 1500
-Wire Wire Line
-	5700 1500 5850 1500
+	6000 1400 6000 1200
 Text GLabel 5150 1800 0    50   Input ~ 0
 TX3.3V
 Text GLabel 5150 1900 0    50   Input ~ 0
 RX3.3V
-Text GLabel 5750 1800 2    50   Input ~ 0
+Text GLabel 5950 1800 2    50   Input ~ 0
 TX5V
-Text GLabel 5750 1900 2    50   Input ~ 0
+Text GLabel 5950 1900 2    50   Input ~ 0
 RX5V
-Wire Wire Line
-	5750 1800 5700 1800
-Wire Wire Line
-	5750 1900 5700 1900
-Wire Wire Line
-	5200 1800 5150 1800
-Wire Wire Line
-	5200 1900 5150 1900
 Text GLabel 14750 4550 1    50   Input ~ 0
 SCK
@@
 F 0 "J11" H 12030 3042 50  0000 L CNN
 F 1 "Conn_01x04" H 12030 2951 50  0000 L CNN
-F 2 "Connector_JST:JST_EH_S04B-EH_1x04_P2.50mm_Horizontal" H 11950 3050 50  0001 C CNN
+F 2 "Connector_JST:JST_EH_B04B-EH-A_1x04_P2.50mm_Vertical" H 11950 3050 50  0001 C CNN
 F 3 "~" H 11950 3050 50  0001 C CNN
 	1    11950 3050
@@
 F 0 "J9" V 10517 7046 50  0000 C CNN
 F 1 "Conn_01x16" V 10426 7046 50  0000 C CNN
-F 2 "Connector_JST:JST_EH_S16B-EH_1x16_P2.50mm_Horizontal" H 10300 7100 50  0001 C CNN
+F 2 "Connector_JST:JST_EH_B16B-EH-A_1x16_P2.50mm_Vertical" H 10300 7100 50  0001 C CNN
 F 3 "~" H 10300 7100 50  0001 C CNN
 	1    10300 7100
@@
 F 0 "J13" H 12250 4850 50  0000 L CNN
 F 1 "Conn_01x08" H 12200 4750 50  0000 L CNN
-F 2 "Connector_JST:JST_EH_S08B-EH_1x08_P2.50mm_Horizontal" H 12100 4750 50  0001 C CNN
+F 2 "Connector_JST:JST_EH_B08B-EH-A_1x08_P2.50mm_Vertical" H 12100 4750 50  0001 C CNN
 F 3 "~" H 12100 4750 50  0001 C CNN
 	1    12100 4750
@@
 F 0 "J8" H 10080 4692 50  0000 L CNN
 F 1 "Conn_01x08" H 10080 4601 50  0000 L CNN
-F 2 "Connector_JST:JST_EH_S08B-EH_1x08_P2.50mm_Horizontal" H 10000 4700 50  0001 C CNN
+F 2 "Connector_JST:JST_EH_B08B-EH-A_1x08_P2.50mm_Vertical" H 10000 4700 50  0001 C CNN
 F 3 "~" H 10000 4700 50  0001 C CNN
 	1    10000 4700
@@
 NoConn ~ 10400 7300
 NoConn ~ 10500 7300
-NoConn ~ 5200 1600
-NoConn ~ 5200 1700
-NoConn ~ 5700 1700
-NoConn ~ 5700 1600
 Text GLabel 15350 2900 2    50   Input ~ 0
 NEXT
@@
 Wire Notes Line
 	9150 8350 9150 6750
+$Comp
+L LEEVAWNS:SHIFT_LEVEL_3.3V_5V U6
+U 1 1 5B71A2E8
+P 5250 1400
+F 0 "U6" H 5550 1625 50  0000 C CNN
+F 1 "SHIFT_LEVEL_3.3V_5V" H 5550 1534 50  0000 C CNN
+F 2 "LEEVAWNS:SHIFTLEVEL" H 5250 1400 50  0001 C CNN
+F 3 "" H 5250 1400 50  0001 C CNN
+	1    5250 1400
+	1    0    0    -1
+$EndComp
+Wire Wire Line
+	5050 1400 5250 1400
+Wire Wire Line
+	5000 1500 5250 1500
+Wire Wire Line
+	5150 1800 5250 1800
+Wire Wire Line
+	5150 1900 5250 1900
+Wire Wire Line
+	5850 1900 5950 1900
+Wire Wire Line
+	5850 1800 5950 1800
+Wire Wire Line
+	5850 1500 6050 1500
+Wire Wire Line
+	5850 1400 6000 1400
+NoConn ~ 5850 1600
+NoConn ~ 5850 1700
+NoConn ~ 5250 1700
+NoConn ~ 5250 1600
 $EndSCHEMATC

Commit message: initilize pcb layout
Parts:
- renumbered J11 to J10, J12 to J11, J13 to J12, J14 to J13, J15 to J14, J6 to J5, J7 to J6, J8 to J7, J9 to J8, J10 to J9, P2 to P1, P3 to P2, P4 to P3, P1 to P4, U2 to U1, U1 to U2, U6 to U4, U4 to U5, U5 to U6

Commit message: repairt schematic, layout pcb
Parts:
- removed J5, J6: Conn_01x06, Connector_JST:JST_EH_B06B-EH-A_1x06_P2.50mm_Vertical, symbol Connector_Generic:Conn_01x06
- Q3: footprint Package_TO_SOT_THT:TO-92_Inline -> Package_TO_SOT_SMD:SOT-23
- renumbered J12 to J10, J13 to J11, J14 to J12, J7 to J5, J8 to J6, J9 to J7, J10 to J8, J11 to J9
Connections:
- net labels removed: SC3, SC4
- wire segments 531 -> 517

Commit message: modifier pcb and schematic net list
Parts:
- J11, J12: footprint Connector_Wire:SolderWirePad_1x02_P5.08mm_Drill1.5mm -> LEEVAWNS:SolderWirePad_1x02_P5.08mm_Drill1.5mm
- renumbered C15 to C13, C16 to C14, C17 to C15, C18 to C16, C19 to C17, C20 to C18, C21 to C19, C22 to C20, C13 to C21, C14 to C22, J9 to J10, J10 to J6, J6 to J8, J8 to J9

Commit message: wiring pcb outline
Connections:
- wire segments 517 -> 514
Changed lines of the file:
@@
 Connection ~ 10900 4600
 Wire Wire Line
-	10900 5100 10900 5050
-Wire Wire Line
-	11100 5050 10900 5050
-Connection ~ 10900 5050
-Wire Wire Line
-	10900 5050 10900 5000
-Wire Wire Line
 	11100 4400 11100 4850
 Wire Wire Line
 	11050 4850 11100 4850
-Connection ~ 11100 4850
-Wire Wire Line
-	11100 4850 11100 5050
 $Comp
 L Device:R R18
@@
 NoConn ~ 14850 1200
 NoConn ~ 14850 1300
+Wire Wire Line
+	10900 5000 10900 5100
 $EndSCHEMATC
