File: PCV MATOME MAIN V5-KICAD 5.0/PCV MATOME MAIN V5-KICAD 5.0.sch (KiCad schematic (older format))
At the start: 88 parts, among them J1 Conn_02x08_Odd_Even, J10 Conn_01x08, J11 Conn_01x02, J12 Conn_01x02, J2 Conn_02x08_Odd_Even, J3 Conn_01x06, J4 Conn_01x06, J5 Conn_01x08, J6 Conn_01x08, J7 Conn_01x02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

Commit message: modified pcb 18/08/2018, test pcb final befor release
Connections:
- net labels added: 3.3VDD, SCL1, SDA1
- net labels removed: GNDPWR
- wire segments 514 -> 591
- no-connect marks 66 -> 67
