File: PCB JIGU MATOME/JIGU MATOME/JIGU MATOME.kicad_pcb (KiCad board)
At the start: 2 copper layers, 7 parts, among them J1 Conn_01x04, J2 Conn_01x04, J3 Conn_01x04, J4 Conn_01x04, J5 Conn_01x08, J6 Conn_01x06, U1 757BS

Commit message: modifier pcb jigu
Parts:
- moved J3 10.5 mm to (131.2, 88.0), turned to 270 degrees
- moved J1 4.53 mm to (123.8, 95.5), turned to 90 degrees
- moved J6 4.26 mm to (160.8, 93.0)
- moved U1 3.95 mm to (142.2, 99.0)
- moved J5 3.75 mm to (153.5, 90.5)
- moved J2 3.29 mm to (123.8, 110.0)
- moved J4 3.29 mm to (131.2, 102.5)
Routing:
- net Net-(J6-Pad5): track 0.00 -> 42.9 mm
- net Net-(J6-Pad6): track 0.00 -> 24.4 mm
- net Net-(J6-Pad3): track 0.00 -> 23.2 mm
- net Net-(J5-Pad2): track 0.00 -> 16.6 mm
- net Net-(J5-Pad3): track 0.00 -> 16.2 mm
- net Net-(J5-Pad4): track 0.00 -> 16.1 mm
- net Net-(J5-Pad6): track 0.00 -> 16.1 mm
- net Net-(J6-Pad2): track 0.00 -> 15.9 mm
- net Net-(J6-Pad4): track 0.00 -> 15.8 mm
- net Net-(J5-Pad7): track 0.00 -> 8.60 mm
- net Net-(J5-Pad5): track 0.00 -> 8.59 mm
- net Net-(J5-Pad8): track 0.00 -> 8.54 mm
- net Net-(J2-Pad4): track 0.00 -> 7.50 mm
- net Net-(J2-Pad3): track 0.00 -> 7.50 mm
- net Net-(J2-Pad2): track 0.00 -> 7.50 mm
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Other:
- board outline added: 45 x 36 mm
- net class SIG added: clearance 0.25, trace_width 0.3, via_dia 1, via_drill 0.5

Commit message: modifier pcb carled
Routing:
- net Net-(J6-Pad5): track 42.9 -> 41.6 mm
- net Net-(J6-Pad3): track 23.2 -> 22.5 mm
- added copper zone on B.Cu, net (none)
- added copper zone on F.Cu, net (none)
Other:
- net class Default: via_dia 0.8 -> 1; via_drill 0.4 -> 0.5
- board text added: "JIGU HOUSING MATOME"
- board text added: "V1 by LEEVAWNS"

Commit message: update
Other:
- board text added: "V1.00"
- board text removed: "V1 by LEEVAWNS"
Changed lines of the file:
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@@
   (page A4)
   (layers
-    (0 F.Cu signal hide)
+    (0 F.Cu signal)
     (31 B.Cu signal)
     (32 B.Adhes user)
@@
   )
   (target plus (at 119.75 117) (size 5) (width 0.15) (layer Edge.Cuts))
-  (gr_text "V1 by LEEVAWNS" (at 150.25 115.5) (layer F.SilkS)
+  (gr_text V1.00 (at 145.5 115.5) (layer F.SilkS)
     (effects (font (size 1.1 1.1) (thickness 0.2)))
   )
@@
   (segment (start 153.5 93) (end 150.75 93) (width 0.3) (layer F.Cu) (net 9))
   (segment (start 150.75 93) (end 148.75 91) (width 0.3) (layer F.Cu) (net 9))
+  (segment (start 148.9 93.9) (end 150.5 95.5) (width 0.3) (layer F.Cu) (net 10))
   (segment (start 150.5 95.5) (end 153.5 95.5) (width 0.3) (layer F.Cu) (net 10))
-  (segment (start 149.027999 94.027999) (end 150.5 95.5) (width 0.3) (layer F.Cu) (net 10))
-  (segment (start 144.222001 94.027999) (end 149.027999 94.027999) (width 0.3) (layer F.Cu) (net 10))
+  (segment (start 144.35 93.9) (end 148.9 93.9) (width 0.3) (layer F.Cu) (net 10))
   (segment (start 138.44 95.19) (end 143.06 95.19) (width 0.3) (layer F.Cu) (net 10))
-  (segment (start 143.06 95.19) (end 144.222001 94.027999) (width 0.3) (layer F.Cu) (net 10))
+  (segment (start 143.06 95.19) (end 144.35 93.9) (width 0.3) (layer F.Cu) (net 10))
   (segment (start 150.25 98) (end 153.5 98) (width 0.3) (layer F.Cu) (net 11))
-  (segment (start 148.817999 96.567999) (end 150.25 98) (width 0.3) (layer F.Cu) (net 11))
-  (segment (start 144.182001 96.567999) (end 148.817999 96.567999) (width 0.3) (layer F.Cu) (net 11))
+  (segment (start 148.7 96.45) (end 150.25 98) (width 0.3) (layer F.Cu) (net 11))
+  (segment (start 144.3 96.45) (end 148.7 96.45) (width 0.3) (layer F.Cu) (net 11))
   (segment (start 138.44 97.73) (end 143.02 97.73) (width 0.3) (layer F.Cu) (net 11))
-  (segment (start 143.02 97.73) (end 144.182001 96.567999) (width 0.3) (layer F.Cu) (net 11))
+  (segment (start 143.02 97.73) (end 144.3 96.45) (width 0.3) (layer F.Cu) (net 11))
   (segment (start 150.5 100.5) (end 153.5 100.5) (width 0.3) (layer F.Cu) (net 12))
   (segment (start 146.06 97.73) (end 147.73 97.73) (width 0.3) (layer F.Cu) (net 12))
   (segment (start 147.73 97.73) (end 150.5 100.5) (width 0.3) (layer F.Cu) (net 12))
   (segment (start 142.44 102.81) (end 138.44 102.81) (width 0.3) (layer F.Cu) (net 13))
-  (segment (start 143.602001 101.647999) (end 142.44 102.81) (width 0.3) (layer F.Cu) (net 13))
-  (segment (start 149.147999 101.647999) (end 143.602001 101.647999) (width 0.3) (layer F.Cu) (net 13))
+  (segment (start 143.7 101.55) (end 142.44 102.81) (width 0.3) (layer F.Cu) (net 13))
+  (segment (start 149.05 101.55) (end 143.7 101.55) (width 0.3) (layer F.Cu) (net 13))
   (segment (start 153.5 103) (end 150.5 103) (width 0.3) (layer F.Cu) (net 13))
-  (segment (start 150.5 103) (end 149.147999 101.647999) (width 0.3) (layer F.Cu) (net 13))
+  (segment (start 150.5 103) (end 149.05 101.55) (width 0.3) (layer F.Cu) (net 13))
   (segment (start 150.5 105.5) (end 153.5 105.5) (width 0.3) (layer F.Cu) (net 14))
   (segment (start 147.75 102.75) (end 150.5 105.5) (width 0.3) (layer F.Cu) (net 14))
@@
   (segment (start 158.25 105.5) (end 157 106.75) (width 0.3) (layer F.Cu) (net 20))
   (segment (start 160.75 105.5) (end 158.25 105.5) (width 0.3) (layer F.Cu) (net 20))
+  (segment (start 147.8 104.05) (end 143.7 104.05) (width 0.3) (layer F.Cu) (net 20))
   (segment (start 157 106.75) (end 150.5 106.75) (width 0.3) (layer F.Cu) (net 20))
-  (segment (start 150.5 106.75) (end 147.937999 104.187999) (width 0.3) (layer F.Cu) (net 20))
-  (segment (start 147.937999 104.187999) (end 143.562001 104.187999) (width 0.3) (layer F.Cu) (net 20))
-  (segment (start 143.562001 104.187999) (end 142.4 105.35) (width 0.3) (layer F.Cu) (net 20))
+  (segment (start 150.5 106.75) (end 147.8 104.05) (width 0.3) (layer F.Cu) (net 20))
+  (segment (start 143.7 104.05) (end 142.4 105.35) (width 0.3) (layer F.Cu) (net 20))
   (zone (net 0) (net_name "") (layer F.Cu) (hatch edge 0.508)
     (connect_pads (clearance 0.508))
