File: PCB MATOME MAIN V5-KICAD 5.0/PCV MATOME MAIN V5-KICAD 5.0.kicad_pcb (KiCad board)
At the start: 2 copper layers, 170 x 95 mm, 88 parts, among them J1 Conn_02x08_Odd_Even, J10 Conn_01x08, J11 Conn_01x02, J12 Conn_01x02, J2 Conn_02x08_Odd_Even, J3 Conn_01x06, J4 Conn_01x06, J5 Conn_01x08, J6 Conn_01x08, J7 Conn_01x02, J8 Conn_01x16, J9 Conn_01x04, P1 Power, P10 CONN_01X01, P11 CONN_01X01, P12 CONN_01X01, P13 CONN_01X01, P2 Analog, P3 Analog, P4 Digital, P5 PWM, P6 PWM, P7 Communication, P8 CONN_01X01, P9 CONN_01X01, Q1 BSS138, Q2 BSS138, Q3 2SC1815, SW1 SW_Push, U1 MAX7219, U2 ESP-12F, U3 MAX7219, U4 SHIFT_LEVEL_3.3V_5V, U5 LM1117-3.3, U6 LD1117S50TR_SOT223

Commit message: fix library
Other:
- rule pad_to_mask_clearance: 0 -> 0.1
Changed lines of the file:
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@@
   )
   (layers
-    (0 F.Cu signal hide)
+    (0 F.Cu signal)
     (31 B.Cu signal)
     (32 B.Adhes user)
@@
     (pad_size 4.064 4.064)
     (pad_drill 3.048)
-    (pad_to_mask_clearance 0)
+    (pad_to_mask_clearance 0.1)
     (aux_axis_origin 103.378 121.666)
     (visible_elements 7FFFFFFF)

Commit message: update
Parts:
- moved C26 0.22 mm to (108.1, 127.5)
Routing:
- net SW11: track 63.3 -> 61.9 mm
- net SW12: track 52.9 -> 51.9 mm
